Commit message: controller issues

File: src/rofous_description/urdf/multirotor_base.xacro (robot description, xacro)
@@ -1,134 +1,115 @@
 <?xml version="1.0"?>
 <!--
-  Copyright 2015 Fadri Furrer, ASL, ETH Zurich, Switzerland
-  Copyright 2015 Michael Burri, ASL, ETH Zurich, Switzerland
-  Copyright 2015 Mina Kamel, ASL, ETH Zurich, Switzerland
-  Copyright 2015 Janosch Nikolic, ASL, ETH Zurich, Switzerland
-  Copyright 2015 Markus Achtelik, ASL, ETH Zurich, Switzerland
-  Licensed under the Apache License, Version 2.0 (the "License");
-  you may not use this file except in compliance with the License.
-  You may obtain a copy of the License at
-  http://www.apache.org/licenses/LICENSE-2.0
-  Unless required by applicable law or agreed to in writing, software
-  distributed under the License is distributed on an "AS IS" BASIS,
-  WITHOUT WARRANTIES OR CONDITIONS OF ANY KIND, either express or implied.
-  See the License for the specific language governing permissions and
-  limitations under the License.
+	Copyright 2015 Fadri Furrer, ASL, ETH Zurich, Switzerland
+	Copyright 2015 Michael Burri, ASL, ETH Zurich, Switzerland
+	Copyright 2015 Mina Kamel, ASL, ETH Zurich, Switzerland
+	Copyright 2015 Janosch Nikolic, ASL, ETH Zurich, Switzerland
+	Copyright 2015 Markus Achtelik, ASL, ETH Zurich, Switzerland
+	Licensed under the Apache License, Version 2.0 (the "License");
+	you may not use this file except in compliance with the License.
+	You may obtain a copy of the License at
+	http://www.apache.org/licenses/LICENSE-2.0
+	Unless required by applicable law or agreed to in writing, software
+	distributed under the License is distributed on an "AS IS" BASIS,
+	WITHOUT WARRANTIES OR CONDITIONS OF ANY KIND, either express or implied.
+	See the License for the specific language governing permissions and
+	limitations under the License.
 -->
 <robot xmlns:xacro="http://ros.org/wiki/xacro">
-  <!-- Macro for the inertia of a box -->
-  <xacro:macro name="box_inertia" params="x y z mass">
-    <inertia ixx="${0.0833333 * mass * (y*y + z*z)}" ixy="0.0" ixz="0.0"
-      iyy="${0.0833333 * mass * (x*x + z*z)}" iyz="0.0"
-      izz="${0.0833333 * mass * (x*x + y*y)}" />
-  </xacro:macro>
-  <!-- Macro for the inertial properties of a box -->
-  <xacro:macro name="box_inertial" params="x y z mass *origin">
-    <inertial>
-      <mass value="${mass}" />
-      <xacro:insert_block name="origin" />
-      <xacro:box_inertia x="${x}" y="${y}" z="${z}" mass="${mass}" />
-    </inertial>
-  </xacro:macro>
-  <!-- Main multirotor link -->
-  <xacro:macro name="multirotor_base_macro"
-    params="robot_namespace mass body_width body_height use_mesh_file mesh_file *inertia">
-    <link name="${robot_namespace}/base_link"></link>
-    <joint name="${robot_namespace}/base_joint" type="fixed">
-      <origin xyz="0 0 0" rpy="0 0 0" />
-      <parent link="${robot_namespace}/base_link" />
-      <child link="${robot_namespace}/base_link_inertia" />
-    </joint>
-    <link name="${robot_namespace}/base_link_inertia">
-      <inertial>
-        <mass value="${mass}" />  <!-- [kg] -->
-        <origin xyz="0 0 0" />
-        <xacro:insert_block name="inertia" />
-      </inertial>
-      <visual>
-        <origin xyz="0 0 0" rpy="0 0 0" />
-        <geometry>
-          <xacro:if value="${use_mesh_file}">
-            <mesh filename="${mesh_file}" scale="1 1 1" />
-          </xacro:if>
-          <xacro:unless value="${use_mesh_file}">
-            <box size="${body_width} ${body_width} ${body_height}"/> <!-- [m] [m] [m] -->
-          </xacro:unless>
-        </geometry>
-      </visual>
-      <collision>
-        <origin xyz="0 0 0" rpy="0 0 0" />
-        <geometry>
-          <box size="${body_width} ${body_width} ${body_height}" /> <!-- [m] [m] [m] -->
-        </geometry>
-      </collision>
-    </link>
-    <!-- attach multirotor_base_plugin to the base_link -->
-    <gazebo>
-      <plugin filename="librofous_gazebo_plugins.so" name="rofous_gazebo_plugins">
-        <robotNamespace>${robot_namespace}</robotNamespace>
-        <linkName>${robot_namespace}/base_link</linkName>
-        <rotorVelocitySlowdownSim>${rotor_velocity_slowdown_sim}</rotorVelocitySlowdownSim>
-      </plugin>
-    </gazebo>
-  </xacro:macro>
-  <!-- Rotor joint and link -->
-  <xacro:macro name="vertical_rotor"
-    params="robot_namespace suffix direction motor_constant moment_constant parent mass_rotor radius_rotor time_constant_up time_constant_down max_rot_velocity motor_number rotor_drag_coefficient rolling_moment_coefficient color use_own_mesh mesh *origin *inertia">
-    <joint name="${robot_namespace}/rotor_${motor_number}_joint" type="continuous">
-      <xacro:insert_block name="origin" />
-      <axis xyz="0 0 1" />
-      <!-- TODO(ff): not currently set because it's not yet supported -->
-      <!-- <limit effort="2000" velocity="${max_rot_velocity}" /> -->
-      <parent link="${parent}" />
-      <child link="${robot_namespace}/rotor_${motor_number}" />
-    </joint>
-    <link name="${robot_namespace}/rotor_${motor_number}">
-      <inertial>
-        <mass value="${mass_rotor}" /> <!-- [kg] -->
-        <xacro:insert_block name="inertia" />
-      </inertial>
-      <visual>
-        <geometry>
-          <!-- <cylinder length="0.005" radius="${radius_rotor}"/> --> <!-- [m] -->
-          <xacro:if value="${use_own_mesh}">
-            <mesh filename="${mesh}"
-              scale="1 1 1" />
-          </xacro:if>
-          <xacro:unless value="${use_own_mesh}">
-            <mesh filename="package://rofous_description/meshes/propeller_${direction}.dae"
-              scale="${radius_rotor} ${radius_rotor} ${radius_rotor}" /> <!-- The propeller meshes have a radius of 1m -->
-            <!-- <box size="${2*radius_rotor} 0.01 0.005"/> -->
-          </xacro:unless>
-        </geometry>
-      </visual>
-      <collision>
-        <geometry>
-          <cylinder length="0.005" radius="${radius_rotor}" /> <!-- [m] -->
-        </geometry>
-      </collision>
-    </link>
-    <gazebo>
-      <plugin name="${robot_namespace}_${suffix}_motor_model" filename="librotors_gazebo_motor_model.so">
-        <robotNamespace>${robot_namespace}</robotNamespace>
-        <jointName>${robot_namespace}/rotor_${motor_number}_joint</jointName>
-        <linkName>${robot_namespace}/rotor_${motor_number}</linkName>
-        <turningDirection>${direction}</turningDirection>
-        <timeConstantUp>${time_constant_up}</timeConstantUp>
-        <timeConstantDown>${time_constant_down}</timeConstantDown>
-        <maxRotVelocity>${max_rot_velocity}</maxRotVelocity>
-        <motorConstant>${motor_constant}</motorConstant>
-        <momentConstant>${moment_constant}</momentConstant>
-        <commandSubTopic>gazebo/command/motor_speed</commandSubTopic>
-        <motorNumber>${motor_number}</motorNumber>
-        <rotorDragCoefficient>${rotor_drag_coefficient}</rotorDragCoefficient>
-        <rollingMomentCoefficient>${rolling_moment_coefficient}</rollingMomentCoefficient>
-        <motorSpeedPubTopic>motor_speed/${motor_number}</motorSpeedPubTopic>
-        <rotorVelocitySlowdownSim>${rotor_velocity_slowdown_sim}</rotorVelocitySlowdownSim>
-      </plugin>
-    </gazebo>
-    <gazebo reference="${robot_namespace}/rotor_${motor_number}">
-      <material>Gazebo/${color}</material>
-    </gazebo>
-  </xacro:macro>
+	<!-- Macro for the inertia of a box -->
+	<xacro:macro name="box_inertia" params="x y z mass">
+		<inertia ixx="${0.0833333 * mass * (y*y + z*z)}" ixy="0.0" ixz="0.0"
+			iyy="${0.0833333 * mass * (x*x + z*z)}" iyz="0.0"
+			izz="${0.0833333 * mass * (x*x + y*y)}" />
+	</xacro:macro>
+	<!-- Macro for the inertial properties of a box -->
+	<xacro:macro name="box_inertial" params="x y z mass *origin">
+		<inertial>
+			<mass value="${mass}" />
+			<xacro:insert_block name="origin" />
+			<xacro:box_inertia x="${x}" y="${y}" z="${z}" mass="${mass}" />
+		</inertial>
+	</xacro:macro>
+	<!-- Main multirotor link -->
+	<xacro:macro name="multirotor_base_macro"
+		params="robot_namespace mass body_width body_height use_mesh_file mesh_file *inertia">
+		<link name="${robot_namespace}/base_link"></link>
+		<joint name="${robot_namespace}/base_joint" type="fixed">
+			<origin xyz="0 0 0" rpy="0 0 0" />
+			<parent link="${robot_namespace}/base_link" />
+			<child link="${robot_namespace}/base_link_inertia" />
+		</joint>
+		<link name="${robot_namespace}/base_link_inertia">
+			<inertial>
+				<mass value="${mass}" />  <!-- [kg] -->
+				<origin xyz="0 0 0" />
+				<xacro:insert_block name="inertia" />
+			</inertial>
+			<visual>
+				<origin xyz="0 0 0" rpy="0 0 0" />
+				<geometry>
+					<xacro:if value="${use_mesh_file}">
+						<mesh filename="${mesh_file}" scale="1 1 1" />
+					</xacro:if>
+					<xacro:unless value="${use_mesh_file}">
+						<box size="${body_width} ${body_width} ${body_height}"/> <!-- [m] [m] [m] -->
+					</xacro:unless>
+				</geometry>
+			</visual>
+			<collision>
+				<origin xyz="0 0 0" rpy="0 0 0" />
+				<geometry>
+					<box size="${body_width} ${body_width} ${body_height}" /> <!-- [m] [m] [m] -->
+				</geometry>
+			</collision>
+		</link>
+		<!-- attach multirotor_base_plugin to the base_link -->
+		<gazebo>
+			<plugin filename="librofous_gazebo_plugins.so" name="rofous_gazebo_plugins">
+				<robotNamespace>${robot_namespace}</robotNamespace>
+				<linkName>${robot_namespace}/base_link</linkName>
+				<rotorVelocitySlowdownSim>${rotor_velocity_slowdown_sim}</rotorVelocitySlowdownSim>
+			</plugin>
+		</gazebo>
+	</xacro:macro>
+	<!-- Rotor joint and link -->
+	<xacro:macro name="vertical_rotor"
+		params="robot_namespace suffix direction motor_constant moment_constant parent mass_rotor radius_rotor time_constant_up time_constant_down max_rot_velocity motor_number rotor_drag_coefficient rolling_moment_coefficient color use_own_mesh mesh *origin *inertia">
+		<joint name="rotor_${motor_number}_joint" type="continuous">
+			<xacro:insert_block name="origin" />
+			<axis xyz="0 0 1" />
+			<!-- TODO(ff): not currently set because it's not yet supported -->
+			<!-- <limit effort="2000" velocity="${max_rot_velocity}" /> -->
+			<parent link="${parent}" />
+			<child link="rotor_${motor_number}" />
+		</joint>
+		<link name="rotor_${motor_number}">
+			<inertial>
+				<mass value="${mass_rotor}" /> <!-- [kg] -->
+				<xacro:insert_block name="inertia" />
+			</inertial>
+			<visual>
+				<geometry>
+					<!-- <cylinder length="0.005" radius="${radius_rotor}"/> --> <!-- [m] -->
+					<xacro:if value="${use_own_mesh}">
+						<mesh filename="${mesh}"
+							scale="1 1 1" />
+					</xacro:if>
+					<xacro:unless value="${use_own_mesh}">
+						<mesh filename="package://rofous_description/meshes/propeller_${direction}.dae"
+							scale="${radius_rotor} ${radius_rotor} ${radius_rotor}" /> <!-- The propeller meshes have a radius of 1m -->
+						<!-- <box size="${2*radius_rotor} 0.01 0.005"/> -->
+					</xacro:unless>
+				</geometry>
+			</visual>
+			<collision>
+				<geometry>
+					<cylinder length="0.005" radius="${radius_rotor}" /> <!-- [m] -->
+				</geometry>
+			</collision>
+		</link>
+		<gazebo reference="rotor_${motor_number}">
+			<material>Gazebo/${color}</material>
+		</gazebo>
+	</xacro:macro>
 </robot>

Commit message: gazebo changes

File: src/rofous_description/urdf/hummingbird.xacro (robot description, xacro)
@@ -16,10 +16,10 @@
   limitations under the License.
 -->
-<robot name="rofous" xmlns:xacro="http://ros.org/wiki/xacro">
+<robot name="hummingbird" xmlns:xacro="http://ros.org/wiki/xacro">
   <!-- Properties (Taken from Novel Dynamic Inversion Architecture Design
 for Quadrocopter Control by Jian Wang et al.) -->
-  <xacro:property name="namespace" value="$(arg namespace)" />
+  <xacro:property name="namespace" value="hummingbird"/>
   <xacro:property name="rotor_velocity_slowdown_sim" value="10" />
-  <xacro:property name="use_mesh_file" value="true" />
+  <xacro:property name="use_mesh_file" value="true"/>
   <xacro:property name="mesh_file" value="package://rofous_description/meshes/hummingbird.dae" />
   <xacro:property name="mass" value="0.68" /> <!-- [kg] -->
@@ -57,4 +57,8 @@
     <xacro:insert_block name="body_inertia" />
   </xacro:multirotor_base_macro>
+  <gazebo>
+    <plugin name="gazebo_ros_control" filename="libgazebo_ros_control.so">
+    </plugin>
+  </gazebo>
   <!-- Instantiate rotors -->
   <xacro:vertical_rotor

File: src/rofous_description/urdf/multirotor_base.xacro (robot description, xacro)
@@ -65,5 +65,5 @@
     </link>
     <!-- attach multirotor_base_plugin to the base_link -->
-    <gazebo>
+<!--     <gazebo>
       <plugin filename="librofous_gazebo_plugins.so" name="rofous_gazebo_plugins">
         <robotNamespace>${robot_namespace}</robotNamespace>
@@ -71,10 +71,19 @@
         <rotorVelocitySlowdownSim>${rotor_velocity_slowdown_sim}</rotorVelocitySlowdownSim>
       </plugin>
-    </gazebo>
+    </gazebo> -->
+  </xacro:macro>
+    <xacro:macro name="EffortTransmission" params="joint n">
+    <transmission name="transmission_${n}">
+      <type>transmission_interface/SimpleTransmission</type>
+      <joint name="${joint}">
+        <hardwareInterface>hardware_interface/EffortJointInterface</hardwareInterface>
+      </joint>
+      <actuator name="motor${n}"/>
+    </transmission>
   </xacro:macro>
   <!-- Rotor joint and link -->
   <xacro:macro name="vertical_rotor"
     params="robot_namespace suffix direction motor_constant moment_constant parent mass_rotor radius_rotor time_constant_up time_constant_down max_rot_velocity motor_number rotor_drag_coefficient rolling_moment_coefficient color use_own_mesh mesh *origin *inertia">
-    <joint name="${robot_namespace}/rotor_${motor_number}_joint" type="continuous">
+    <joint name="rotor_${motor_number}_joint" type="continuous">
       <xacro:insert_block name="origin" />
       <axis xyz="0 0 1" />
@@ -82,7 +91,7 @@
       <!-- <limit effort="2000" velocity="${max_rot_velocity}" /> -->
       <parent link="${parent}" />
-      <child link="${robot_namespace}/rotor_${motor_number}" />
+      <child link="rotor_${motor_number}" />
     </joint>
-    <link name="${robot_namespace}/rotor_${motor_number}">
+    <link name="rotor_${motor_number}">
       <inertial>
         <mass value="${mass_rotor}" /> <!-- [kg] -->
@@ -109,5 +118,6 @@
       </collision>
     </link>
-    <gazebo>
+    <xacro:EffortTransmission n="${motor_number}" joint="rotor_${motor_number}_joint" />
+    <!-- <gazebo>
       <plugin name="${robot_namespace}_${suffix}_motor_model" filename="librotors_gazebo_motor_model.so">
         <robotNamespace>${robot_namespace}</robotNamespace>
@@ -130,5 +140,5 @@
     <gazebo reference="${robot_namespace}/rotor_${motor_number}">
       <material>Gazebo/${color}</material>
-    </gazebo>
+    </gazebo> -->
   </xacro:macro>
 </robot>
