Commit message: mornin push

File: dysepy/data/robots/penguin/robot.xacro (robot description, xacro)
@@ -9,5 +9,5 @@
   <xacro:property name="pi_value" value="3.14159263" />
   <xacro:property name="radiusp" value="0.20" />
-  <xacro:property name="prop_loc" value="0.15909" />
+  <xacro:property name="prop_loc" value="0.2" />
 <!-- ======================================================== -->
   <xacro:include filename="$(find dysepy)/data/robots/penguin/material.xacro" />
@@ -26,32 +26,32 @@
   <link name="base_link1">
     <visual>
+      <origin xyz="0 0 0" rpy="0 0 ${pi_value/2}" />
+      <geometry>
+        <box size="${width} ${length} ${height}" />
+      </geometry>
+      <material name="red" />
+    </visual>
+    <collision>
       <origin xyz="0 0 0" rpy="0 0 ${pi_value/4}" />
       <geometry>
         <box size="${width} ${length} ${height}" />
       </geometry>
-      <material name="red" />
-    </visual>
-    <collision>
-      <origin xyz="0 0 0" rpy="0 0 ${pi_value/4}" />
+    </collision>
+    <xacro:default_inertial mass="${mass_fr}" p="${pi_value/4}" ix_value="${0.04989/2}" iy_value="${0.04989/2}" iz_value="${0.24057/2}" />
+  </link>
+<!-- ======================================================== -->
+  <link name="base_link2">
+    <visual>
+      <origin xyz="0 0 0" rpy="0 0 0" />
       <geometry>
         <box size="${width} ${length} ${height}" />
       </geometry>
-    </collision>
-    <xacro:default_inertial mass="${mass_fr}" p="${pi_value/4}" ix_value="${0.04989/2}" iy_value="${0.04989/2}" iz_value="${0.24057/2}" />
-  </link>
-<!-- ======================================================== -->
-  <link name="base_link2">
-    <visual>
-      <origin xyz="0 0 0" rpy="0 0 ${-pi_value/4}" />
+      <material name="white" />
+    </visual>
+    <collision>
+      <origin xyz="0 0 0" rpy="0 0 0" />
       <geometry>
         <box size="${width} ${length} ${height}" />
       </geometry>
-      <material name="white" />
-    </visual>
-    <collision>
-      <origin xyz="0 0 0" rpy="0 0 ${-pi_value/4}" />
-      <geometry>
-        <box size="${width} ${length} ${height}" />
-      </geometry>
     </collision>
     <xacro:default_inertial mass="${mass_fr}" p="${-pi_value/4}" ix_value="${0.04989/2}" iy_value="${0.04989/2}" iz_value="${0.24057/2}" />
@@ -60,5 +60,5 @@
   <link name="plate1">
     <visual>
-      <origin xyz="0 0 0" rpy="0 0 0" />
+      <origin xyz="0 0 0" rpy="0 0 ${pi_value}" />
       <geometry>
         <box size="${0.12} ${0.12} ${0.01}" />
@@ -67,5 +67,5 @@
     </visual>
     <collision>
-      <origin xyz="0 0 0" rpy="0 0 0" />
+      <origin xyz="0 0 0" rpy="0 0 ${pi_value}" />
       <geometry>
         <box size="${0.12} ${0.12} ${0.01}" />
@@ -271,5 +271,5 @@
     <parent link="base_link2" />
     <child link="prop_front_right" />
-    <origin xyz="${prop_loc - 0.01} ${prop_loc - 0.01} 0.021" rpy="0 0 0"/>
+    <origin xyz="${prop_loc - 0.01} 0 0.021" rpy="0 0 0"/>
     <axis xyz="0 0 1" />
   </joint>
@@ -279,5 +279,5 @@
     <parent link="base_link1" />
     <child link="prop_front_left" />
-    <origin xyz="${-prop_loc + 0.01} ${prop_loc - 0.01} 0.021" rpy="0 0 0" />
+    <origin xyz="0 ${prop_loc - 0.01} 0.021" rpy="0 0 0" />
     <axis xyz="0 0 1" />
   </joint>
@@ -287,5 +287,5 @@
     <parent link="base_link1" />
     <child link="prop_back_right" />
-    <origin xyz="${prop_loc - 0.01} ${-prop_loc + 0.01} 0.021" rpy="0 0 0" />
+    <origin xyz="0 ${-prop_loc + 0.01} 0.021" rpy="0 0 0" />
     <axis xyz="0 0 1" />
   </joint>
@@ -295,5 +295,5 @@
     <parent link="base_link2" />
     <child link="prop_back_left" />
-    <origin xyz="${-prop_loc + 0.01} ${-prop_loc + 0.01} 0.021" rpy="0 0 0" />
+    <origin xyz="${-prop_loc + 0.01} 0 0.021" rpy="0 0 0" />
     <axis xyz="0 0 1" />
   </joint>
@@ -319,5 +319,5 @@
     <parent link="base_link2" />
     <child link="cyl1" />
-    <origin xyz="${prop_loc - 0.01} ${prop_loc - 0.01} 0.01" rpy="0 0 0" />
+    <origin xyz="${prop_loc - 0.01} 0 0.01" rpy="0 0 0" />
     <axis xyz="0 0 1" />
   </joint>
@@ -327,5 +327,5 @@
     <parent link="base_link2" />
     <child link="cyl2" />
-    <origin xyz="${-prop_loc + 0.01} ${-prop_loc + 0.01} 0.01" rpy="0 0 0" />
+    <origin xyz="0 ${-prop_loc + 0.01} 0.01" rpy="0 0 0" />
     <axis xyz="0 0 1" />
   </joint>
@@ -335,5 +335,5 @@
     <parent link="base_link1" />
     <child link="cyl3" />
-    <origin xyz="${-prop_loc + 0.01} ${prop_loc - 0.01} 0.01" rpy="0 0 0" />
+    <origin xyz="${-prop_loc + 0.01} 0 0.01" rpy="0 0 0" />
     <axis xyz="0 0 1" />
   </joint>
@@ -343,5 +343,5 @@
     <parent link="base_link1" />
     <child link="cyl4" />
-    <origin xyz="${prop_loc - 0.01} ${-prop_loc + 0.01} 0.01" rpy="0 0 0" />
+    <origin xyz="0 ${prop_loc + 0.01} 0.01" rpy="0 0 0" />
     <axis xyz="0 0 1" />
   </joint>

Commit message: updates

File: dysepy/data/robots/penguin/robot.xacro (robot description, xacro)
@@ -9,5 +9,5 @@
   <xacro:property name="pi_value" value="3.14159263" />
   <xacro:property name="radiusp" value="0.20" />
-  <xacro:property name="prop_loc" value="0.2" />
+  <xacro:property name="prop_loc" value="0.23" />
 <!-- ======================================================== -->
   <xacro:include filename="$(find dysepy)/data/robots/penguin/material.xacro" />
