Commit message: save

File: buffpy/data/robots/penguin/robot.xacro (robot description, xacro)
@@ -11,6 +11,6 @@
   <xacro:property name="prop_loc" value="0.23" />
 <!-- ======================================================== -->
-  <xacro:include filename="$(find dysepy)/data/robots/penguin/material.xacro" />
-  <!-- <xacro:include filename="$(find dysepy)/data/robots/penguin/Kwad.gazebo" /> -->
+  <xacro:include filename="$(find buffpy)/data/robots/penguin/material.xacro" />
+  <!-- <xacro:include filename="$(find buffpy)/data/robots/penguin/Kwad.gazebo" /> -->
 <!-- ======================================================== -->
   <!-- Define inertial macro -->
@@ -164,5 +164,5 @@
       <origin xyz="0 0 0" rpy="0 0 0" />
       <geometry>
-        <mesh filename="package://dysepy/data/robots/penguin/22V10.dae" scale="0.005 0.005 0.005" />
+        <mesh filename="package://buffpy/data/robots/penguin/22V10.dae" scale="0.005 0.005 0.005" />
       </geometry>
     </visual>
